File: cytron-motor-driver/cytron-1.sch (EAGLE design)
At the start: 76 parts, among them M2A PUSH_BUTTON, M2B PUSH_BUTTON, T4 2N2222, T5 2N2222, T6 2N2222

Commit message: update motor driver
Parts:
- removed B: (no value), MIA_LIBRARY-2-2-2:ROSTA.POWER
- removed KK1, KK2, KK3, KK4, KK5, KK6, KK7, KK8: HEAT_SINK, MIA_LIBRARY-2-2-2:HEAT_SINK
- removed PWR: (no value), led:LED5MM
- removed Q1, Q2, Q3, Q4: (no value), MIA_LIBRARY-2-2-2:MOSFET_NTO220BV
- removed R6: 1k, rcl8:R-US_0204/7
- removed U$2: DC-DC-STEP-UP-MT3608, MIA_LIBRARY-2-2-2:DC-DC-STEP-UP-MT3608
- added C3: 1nF, MIA_LIBRARY-2-2-2:CAPACITOR
- added C4: 470uf, MIA_LIBRARY-2-2-2:CAP_POL
- added C5: 100n, MIA_LIBRARY-2-2-2:CAPACITOR
- added D13: 1N5817-B, MIA_LIBRARY-2-2-2:DIODE(1A)-PTH
- added IC1: MC34063AP, MIA_LIBRARY-2-2-2:MC34063AP
- added L2: 330uh, MIA_LIBRARY-2-2-2:INDUCTOR-2PIS2816
- added MOTOR: (no value), MIA_LIBRARY-2-2-2:ROSTA.POWER
- added POWER.: LED3MM, MIA_LIBRARY-2-2-2:LED3MM
- added R-1: 1.2k, MIA_LIBRARY-2-2-2:RES-7
- added R-2: 4.4k, MIA_LIBRARY-2-2-2:RES-7
- added R3: 10k, MIA_LIBRARY-2-2-2:TRIM_EU-CA6V
- added R37: RES-7, MIA_LIBRARY-2-2-2:RES-7
- added R4: 100, MIA_LIBRARY-2-2-2:RES-7
- added R5: 56k, MIA_LIBRARY-2-2-2:RES-7
- added R7: 3.3k, MIA_LIBRARY-2-2-2:RES-7
- added U$3: HEAT-SINK, MIA_LIBRARY-2-2-2:HEAT-SINK
- added U$4, U$5: 100u, MIA_LIBRARY-2-2-2:CAP_POL
- 2A, B2: value (none) -> LED3MM; device led:LED3MM -> MIA_LIBRARY-2-2-2:LED3MM
- 3, 4: device irs:IR2184D -> MIA_LIBRARY-2-2-2:IR2184D
- C1, C14, C15, C17, C18, C2, C20, C21, C22: device rcl8:C-US025-025X050 -> MIA_LIBRARY-2-2-2:CAPACITOR
- D10, D5, D6, D7: value 1A/50V/1.1V -> BY396; device MIA_LIBRARY-2-2-2:DIODE(1A)-PTH -> diode:BY396
- D11, D12, D8, D9: value 1N5060GP -> 1A/50V/1.1V; device diode:1N5060GP -> MIA_LIBRARY-2-2-2:DIODE(1A)-PTH
- IC5: device MIA_LIBRARY-2-2-2:78XXL -> MIA_LIBRARY-2-2-2:78XXS
- M2A, M2B: device MIA_LIBRARY (1):PUSH_BUTTON -> MIA_LIBRARY-2-2-2:PUSH_BUTTON
- R21, R22, R23, R24: value 10 -> 220
- T4, T5, T6: value 2N2222 -> TR-2N2222_1; device transistor:2N2222 -> MIA_LIBRARY-2-2-2:TR-2N2222_1; SPICEPREFIX (none) -> J
- U$1: value RES-7 -> HEAT-SINK-10HEAT-SINK-10; device MIA_LIBRARY-2-2-2:RES-7 -> MIA_LIBRARY-2-2-2:HEAT-SINK-10HEAT-SINK-10
Connections:
- removed net N$1: PWR.C, R6.1
- removed net N$6 (its old number): D4.A, Q4.G, Q6.G, R22.1
- new net N$10: D13.A, IC1.SWC, L2.2
- new net N$12: IC1.FB, R-2.2, R3.S, R5.1
- new net N$15: IC1.DC, R4.2
- new net N$16: POWER..A, R7.1
- new net N$19: U$3.PIN2
- new net N$20: U$3.PIN1
- new net N$21: R-1.2, R-2.1
- new net N$5: D4.A, Q6.G, R22.1
- new net N$9: C3.1, IC1.TC
- net +B: now also MAIN-2.KL, U$5.+; no longer KK1.P$1, KK2.P$1, KK5.P$1, KK6.P$1, MAIN-1.KL, Q1.D, Q3.D
- net 12V: now also IC1.IS, IC1.VCC, L2.1, R4.1, U$4.+; no longer U$2.IN+
- net 2A: now also MOTOR-1.KL; no longer B-1.KL, KK7.P$1, KK8.P$1, Q3.S, Q4.D
- net 2B: now also MOTOR-2.KL; no longer B-2.KL, KK3.P$1, KK4.P$1, Q1.S, Q2.D
- net GND: now also C3.2, C4.-, C5.1, IC1.GND, IC1.SWE, MAIN-1.KL, POWER..C, R-1.1, R3.A, U$4.-, U$5.-; no longer MAIN-2.KL, Q2.S, Q4.S, R6.2, U$2.IN-, U$2.OUT-
- net N$25: no longer Q3.G
- net N$32: no longer Q2.G
- net N$33: no longer Q1.G
- net N$40: now also R37.2; no longer U$1.2
- net N$8: now also R37.1; no longer U$1.1
- net VCC: now also C4.+, C5.2, D13.C, R5.2, R7.2; no longer PWR.A, U$2.OUT+
Other:
- moved on the sheet: 3, 4, C1, C14, C15, C16, C17, C18, C19, C2, C20, C21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
